Commit message: Corrección Gazebo

File: urdf/dd_robot.urdf (robot description, URDF)
Before this commit: robot dd_robot, 3 links, 2 joints
Links:
- added link back_wheel, mass 0.025; collision cylinder length=0.01 radius=0.017; visual cylinder length=0.01 radius=0.017
- added link base_footprint
- added link front_wheel, mass 0.025; collision cylinder length=0.01 radius=0.017; visual cylinder length=0.01 radius=0.017
- link base_link: geometry collision cylinder length=0.089 radius=0.175; visual cylinder length=0.089 radius=0.175
Joints:
- added joint fixed_joint: type fixed, parent base_footprint, child base_link, origin xyz=0.0 0.0 0.0575 rpy=0.0 0.0 0.0
- added joint joint_back_wheel: type fixed, parent base_link, child back_wheel, origin xyz=-0.115 0.0 -0.039 rpy=0.0 0.0 0.0
- added joint joint_front_wheel: type fixed, parent base_link, child front_wheel, origin xyz=0.115 0.0 -0.039 rpy=0.0 0.0 0.0
- joint joint_left_wheel: limit effort=10 velocity=6.0 -> effort=100 velocity=6.0; origin xyz=0.0 0.117539 0.03423 rpy=0.0 0.0 0.0 -> xyz=0.0 0.117539 -0.0233 rpy=0.0 0.0 0.0
- joint joint_right_wheel: limit effort=10 velocity=6.0 -> effort=100 velocity=6.0; origin xyz=0.0 -0.117539 0.03423 rpy=0.0 0.0 0.0 -> xyz=0.0 -0.117539 -0.0233 rpy=0.0 0.0 0.0
